File: PCB/robot.kicad_pcb (KiCad board)
At the start: 4 copper layers, 90 x 72 mm, 61 parts, among them J201 Motor_L, J202 bordure_R, J204 LIDAR, J205 Motor_R, J206 BUMPER_F, J207 BUMPER_B, J208 BUMPER_R, J209 BUMPER_L, J210 Conn_02x07_Odd_Even, J211 bordure_F, J401 Conn_BAT, SW202 SW_Push, U201 STM32G070RBTx, U303 ZXBM5210-SP, U304 ZXBM5210-SP, U401 MP1475DJ-LF-P, U402 MIC5317, Y201 16M

Commit message: chore: pcb
Routing:
- net /STM32/VCP_TX: track 69.3 -> 71.0 mm, vias 3 -> 4
- net /STM32/SWCLK: track 43.6 -> 45.2 mm
- net /STM32/NRST: track 73.7 -> 74.9 mm, vias 3 -> 4
- net /STM32/LED_B: track 68.8 -> 70.0 mm
- net /STM32/VCP_RX: track 59.6 -> 60.6 mm
- net /STM32/LIDAR_TX: track 48.8 -> 47.9 mm

Commit message: update: pcb
Parts:
- added G***: LOGO, LOGO, F.Cu at (54.8, 66.5)
- moved C308 1.35 mm to (131.2, 83.2)
Routing:
- net GND: track 0.00 -> 12.2 mm, vias 21 -> 25
- net /STM32/V_BORDURE_F: track 43.9 -> 51.7 mm, vias 1 -> 0
- net /STM32/Endoder_LB: track 54.0 -> 57.1 mm
- net /Motor/FWD_ML: track 55.8 -> 52.7 mm
- net /STM32/BUMPER_R: track 88.8 -> 91.3 mm
- net /Motor/M_R2: track 15.4 -> 16.9 mm
- net /STM32/SWCLK: track 45.2 -> 43.7 mm
- net /STM32/SWDIO: track 43.3 -> 41.8 mm
- net /STM32/BUMPER_F: track 44.5 -> 45.5 mm
- net /Motor/FWD_MR: track 34.9 -> 35.5 mm
- net /Motor/M_L2: track 26.0 -> 26.6 mm
Other:
- board text added: "Clément Dorian Gaël Laksan"
